File: LCD daughter board/LCD_Daughter/LCD_Daughter.kicad_pcb (KiCad board)
At the start: 2 copper layers, 110 x 64 mm, 12 parts, among them J1 JST EH 9pos

Commit message: Renamed SPI busses to match RPI's names. Fixed code to use the correct SPI busses.
Connections:
- net SPI 0 nSS renamed SPI 1 nSS
- net SPI 1 SS SCREEN renamed SPI 0 SS SCREEN
- net SPI 1 SS SD renamed SPI 0 SS SD
- A1 pad 1: SPI 1 MISO -> SPI 0 MISO
- A1 pad 16: SPI 0 MOSI -> SPI 1 MOSI
- A1 pad 19: SPI 0 SCK -> SPI 1 SCK
- A1 pad 20: SPI 0 MISO -> SPI 1 MISO
- A1 pad 4: SPI 1 SCK -> SPI 0 SCK
- A1 pad 5: SPI 1 MOSI -> SPI 0 MOSI
- J1 pad 6: SPI 0 MOSI -> SPI 1 MOSI
- J1 pad 7: SPI 0 SCK -> SPI 1 SCK
- J1 pad 9: SPI 0 MISO -> SPI 1 MISO
- LCD1 pad 16: SPI 1 MOSI -> SPI 0 MOSI
- LCD1 pad 17: SPI 1 MISO -> SPI 0 MISO
- LCD1 pad 18: SPI 1 SCK -> SPI 0 SCK
- LCD1 pad 6: SPI 1 MOSI -> SPI 0 MOSI
- LCD1 pad 7: SPI 1 SCK -> SPI 0 SCK
- LCD1 pad 9: SPI 1 MISO -> SPI 0 MISO
Routing:
- net SPI 1 MISO: track 144.8 -> 50.6 mm
- net SPI 0 MISO: track 50.6 -> 144.8 mm
- net SPI 1 MOSI: track 129.2 -> 50.8 mm, vias 1 -> 0
- net SPI 0 MOSI: track 50.8 -> 129.2 mm, vias 0 -> 1
- net SPI 1 SCK: track 124.4 -> 53.3 mm
- net SPI 0 SCK: track 53.3 -> 124.4 mm
